File: BridgePCB/PiMate300_bridge.kicad_pcb (KiCad board)
At the start: 2 copper layers, 247.3 x 33 mm, 28 parts, among them J1 PI_CON, J2 LEFT_CON, J3 RIGHT_CON, U1 KBD_ROW, U2 CD74HC4067SM, U3 KBD_COL

Commit message: Started work on Right PCB, added model for double stack USB and started positioning.
Connections:
- J2 pad 19: GND -> KBD_EN
- J2 pad 20: GND -> KBD_PWR
- U2 pad 15: +3V3 -> KBD_EN
- U2 pad 24: +3V3 -> KBD_PWR
Routing:
- net KBD_PWR: track 0.00 -> 146.8 mm, vias 0 -> 1
- net KBD_EN: track 0.00 -> 135.5 mm, vias 0 -> 1
- net GND: track 146.5 -> 185.7 mm
- net +3V3: track 210.2 -> 193.7 mm, vias 3 -> 1
- net Net-(J2-Pad49): track 90.3 -> 94.8 mm
- net Net-(J2-Pad45): track 102.3 -> 106.3 mm
- net Net-(J2-Pad47): track 102.7 -> 106.6 mm
- net Net-(J2-Pad41): track 99.4 -> 102.5 mm
- net Net-(J2-Pad43): track 97.9 -> 100.2 mm
