File: LeftPCB/LeftPCB_PWR.sch (KiCad schematic (older format))
At the start: 0 parts

Commit message: Updated schematic for LeftPCB, completed USB hub and Keyboard HID device, and started work on the power supply have the external, 3.3v, and 5v mapped out, just need to figure out battery charging/usage circuits.
Parts:
- added C?: 15uF, symbol Device:C_Small
- added C? (x3): 100nF, symbol Device:C_Small
- added C? (x3): 10uF, symbol Device:C_Small
- added C?: 100pF, symbol Device:C_Small
- added C? (x2): 22uF, symbol Device:C_Small
- added C?: 100nf, symbol Device:C_Small
- added IC?: TPS56637RPAR, TPS56637RPAR, symbol TPS56637RPAR:TPS56637RPAR
- added IC?: TPS62056DGSR, SOP50P490X110-10N, symbol TPS62056DGSR:TPS62056DGSR
- added J?: Power In, symbol Connector:Barrel_Jack_MountingPin
- added L?: L_Small, symbol Device:L_Small
- added L?: 10uH, symbol Device:L_Small
- added L?: 3.3uH, symbol Device:L_Small
- added R?: 191k, symbol Device:R_Small_US
- added R? (x4): 10k, symbol Device:R_Small_US
- added R?: 20k, symbol Device:R_Small_US
- added R?: 54.9k, symbol Device:R_Small_US
- added U?: TPS565208, Package_TO_SOT_SMD:SOT-23-6, symbol Regulator_Switching:TPS565208
Connections:
- new net: C?.2, C?.2, IC?.11 (VIN_2), IC?.12 (VIN_3), IC?.13 (VIN_4), IC?.8 (VIN_1), J?.1
- new net: C?.1, IC?.2 (FB), R?.1, R?.2
- new net: C?.1, IC?.6 (SW), L?.2
- new net: C?.2, IC?.7 (BOOT)
- new net: C?.2, R?.1
- new net: IC?.9 (SW), L?.1
- new net: R?.1, R?.2, U?.1 (GND)
- new net: L?.1, U?.2 (SW)
- new net: R?.1, R?.2, U?.4 (VFB)
- new net: C?.2, U?.6 (VBST)
- new net +12V: C?.1, C?.1, C?.1, C?.2, IC?.1 (VIN), IC?.8 (EN), L?.1, R?.2, R?.2, U?.3 (VIN)
- new net +3V3: C?.1, IC?.5 (FB), L?.2
- new net +5V: C?.1, C?.1, L?.2, R?.2
- new net GND: C?.1, C?.1, C?.1, C?.2, C?.2, C?.2, IC?.10 (MODE), IC?.2 (LBO), IC?.3 (AGND), IC?.3 (GND), IC?.4 (PG), IC?.6 (LBI), IC?.7 (SYNC), IC?.9 (PGND), J?.2, J?.MP (MountPin), R?.1, R?.1, R?.1
- new net GNDPWR: C?.2, C?.2, R?.2
- new net SYS_PWR_EN: U?.5 (EN)
Other:
- note added: "3.3v 800ma Power Supply, Always enabled"
- note added: "5v 5a System Power Supply, enabled by MSP430"
- note added: "Power in from external power supply, output is 12v 5a"
