File: LeftPCB/LeftPCB.kicad_pcb (KiCad board)
At the start: 2 copper layers, 70.9 x 98.5 mm, 128 parts, among them IC1 FE1.1S, IC2 TPS62056DGSR, IC3 BQ40Z60RHBT, J1 Bridge_Conn, J2 Conn_01x05_Male, J3 SMB_CON, J4 BATT_CON, Q1 LODRV, Q2 HIDRV, Q3 ACFET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

Commit message: Updated and performed layout on most of left PCB, still have a few things to add.
Parts:
- removed R27: 1M, Resistors_SMD:R_0603
- added J10: PI_USB3, Pin_Headers:Pin_Header_Straight_1x04_Pitch1.00mm, F.Cu at (61.5, 121.7)
- added J5: PI_USB0, Pin_Headers:Pin_Header_Straight_1x04_Pitch1.00mm, F.Cu at (66.2, 92.9)
- added J6: PI_USB1, Pin_Headers:Pin_Header_Straight_1x04_Pitch1.00mm, F.Cu at (56.4, 121.7)
- added J7: Conn_02x04_Odd_Even, Pin_Headers:Pin_Header_Straight_2x04_Pitch1.00mm, B.Cu at (66.1, 81.2)
- added J8: RJ45, Connectors:RJ45_8, F.Cu at (60.3, 75.3)
- added J9: PI_USB2, Pin_Headers:Pin_Header_Straight_1x04_Pitch1.00mm, F.Cu at (59.0, 121.7)
- C44, C46: moved to B.Cu
- R49: footprint Resistors_SMD:R_0603 -> Resistors_SMD:R_2010; moved to B.Cu
- U2: footprint MSP430F5508IRGCR:QFN50P900X900X100-65N -> Housings_QFP:LQFP-48_7x7mm_Pitch0.5mm
- moved C46 42.7 mm to (62.1, 42.2), turned to 180 degrees
- moved R49 35.7 mm to (93.5, 67.2), turned to 270 degrees
- moved C44 32.2 mm to (95.9, 67.2), turned to 270 degrees
- moved C15 30.3 mm to (109.9, 84.4)
- moved C2 26.3 mm to (65.4, 90.3), turned to 270 degrees
- moved R24 25.9 mm to (109.9, 85.9)
- moved C16 25.6 mm to (109.9, 83.0)
- moved C9 24.7 mm to (59.6, 95.6), turned to 270 degrees
- moved D3 22.8 mm to (57.8, 95.6), turned to 90 degrees
- moved C1 22.7 mm to (64.0, 90.3)
- moved R26 22.6 mm to (74.0, 114.2)
- moved R14 21.1 mm to (57.8, 92.2), turned to 270 degrees
- moved D2 21.0 mm to (53.9, 95.6), turned to 90 degrees
- moved R20 20.4 mm to (115.4, 105.7), turned to 90 degrees
- moved R6 19.0 mm to (61.0, 95.6), turned to 90 degrees
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Connections:
- R18 pad 1: Net-(D6-Pad1) -> GND
- R18 pad 2: GND -> Net-(D6-Pad1)
- R19 pad 1: Net-(D7-Pad1) -> GND
- R19 pad 2: GND -> Net-(D7-Pad1)
- R20 pad 1: Net-(D8-Pad1) -> GND
- R20 pad 2: GND -> Net-(D8-Pad1)
- U2 pad 1: ANALOG_BRIGHTNESS -> Net-(U2-Pad1)
- U2 pad 14: KBD_COL_SEL_0 -> USB_RESET
- U2 pad 15: KBD_COL_SEL_1 -> Net-(U2-Pad15)
- U2 pad 16: KBD_COL_SEL_2 -> IS_PWR_DWN
- U2 pad 17: KBD_COL_SEL_3 -> PI_SHUTDOWN
- U2 pad 18: KBD_COL_VAL -> SYS_PWR_EN
- U2 pad 19: USB_RESET -> KBD_ROW_0
- U2 pad 20: PI_SHUTDOWN -> KBD_ROW_1
- U2 pad 21: IS_PWR_DWN -> KBD_ROW_2
- U2 pad 22: SYS_PWR_EN -> KBD_COL_SEL_1
- U2 pad 23: Net-(U2-Pad23) -> KBD_ROW_3
- U2 pad 24: Net-(D8-Pad2) -> KBD_COL_SEL_0
- U2 pad 25: Net-(D7-Pad2) -> KBD_ROW_4
- U2 pad 26: Net-(D6-Pad2) -> KBD_COL_SEL_3
- U2 pad 29: KBD_ROW_0 -> KBD_ROW_5
- U2 pad 3: Net-(R27-Pad1) -> ANALOG_BRIGHTNESS
- U2 pad 30: KBD_ROW_1 -> KBD_COL_SEL_2
- U2 pad 31: KBD_ROW_2 -> KBD_ROW_6
- U2 pad 32: KBD_ROW_3 -> KBD_COL_VAL
- U2 pad 33: KBD_ROW_4 -> KBD_ROW_7
- U2 pad 34: KBD_ROW_5 -> Net-(D6-Pad2)
- U2 pad 35: KBD_ROW_6 -> Net-(D7-Pad2)
- U2 pad 36: KBD_ROW_7 -> Net-(D8-Pad2)
Routing:
- net +5V: track 0.00 -> 166.6 mm, vias 0 -> 2
- net Net-(R21-Pad2): track 0.00 -> 112.2 mm, vias 0 -> 3
- net HSRN: track 0.00 -> 101.9 mm, vias 0 -> 2
- net KBD_USB_DP: track 0.00 -> 71.2 mm, vias 0 -> 2
- net KBD_USB_DN: track 0.00 -> 68.8 mm, vias 0 -> 2
- net +3V3: track 0.00 -> 61.2 mm, vias 0 -> 10
- net GNDD: track 0.00 -> 59.5 mm, vias 0 -> 2
- net ANALOG_GND: track 0.00 -> 56.6 mm, vias 0 -> 3
- net IS_PWR_DWN: track 0.00 -> 56.0 mm, vias 0 -> 2
- net SYS_PWR_EN: track 0.00 -> 55.8 mm, vias 0 -> 4
- net PI_SHUTDOWN: track 0.00 -> 52.4 mm, vias 0 -> 2
- net Net-(C47-Pad2): track 0.00 -> 52.0 mm, vias 0 -> 2
- net USB_RESET: track 0.00 -> 45.0 mm, vias 0 -> 3
- net Net-(R1-Pad2): track 0.00 -> 41.8 mm, vias 0 -> 4
- net Net-(C11-Pad2): track 0.00 -> 37.8 mm, vias 0 -> 2
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- added copper zone on F.Cu, net +3V3
- added copper zone on B.Cu, net GND
- added copper zone on B.Cu, net GNDS
- added copper zone on F.Cu, net HSRN
- added copper zone on F.Cu, net HSRP
- added copper zone on F.Cu, net Net-(C31-Pad2)
- added copper zone on F.Cu, net Net-(C47-Pad2)
- added copper zone on F.Cu, net Net-(Q4-Pad5)
- added copper zone on F.Cu, net PH
- added copper zone on F.Cu, net VCC
